File: kicad/Onboarding Project kicad/Onboarding Project kicad.kicad_sch (KiCad schematic)
At the start: 0 parts

Commit message: Created KiCad schematic and Python calculations
Parts:
- added C1: 680 pF, Connector_PCBEdge:BUS_PCIexpress_x1, symbol Device:C_Small
- added C2: 100 uF, symbol Device:C_Small
- added C4: 300uF, symbol Device:C_Small
- added D1: 1N5819, Diode_THT:D_DO-41_SOD81_P10.16mm_Horizontal, symbol Diode:1N5819
- added L1:: 220uH, Package_DIP:DIP-8_W7.62mm, symbol Device:L_Small
- added R: 180Ω, symbol Device:R_Small
- added R1: 1kΩ, Diode_THT:D_DO-41_SOD81_P10.16mm_Horizontal, symbol Device:R_Small
- added R2: 18kΩ, symbol Device:R_Small
- added Rsc: 0.22Ω, Package_DIP:DIP-8_W7.62mm, symbol Device:R_Small
- added U1: MC34063AP, Package_DIP:DIP-8_W7.62mm, symbol Regulator_Switching:MC34063AP
Connections:
- new net: C1.1, U1.3 (TC)
- new net: D1.2 (A), L1:.2
- new net: L1:.1, R.1, Rsc.1, U1.7 (Ipk)
- new net: R.2, U1.8 (DC)
- new net: R1.1, R2.2, U1.5 (Vfb)
- new net GND: C1.2, C2.1, C4.1, R1.2, U1.2 (SwE), U1.4 (GND)
- new net Vin: C2.2, Rsc.2, U1.6 (Vin)
- new net Vout: C4.2, D1.1 (K), R2.1, U1.1 (SwC)

Commit message: Update schematic to rev 1.1: fixed pin 1 wiring
Connections:
- net Vout: no longer U1.1 (SwC)
- net at D1.2 (A), L1:.2: now also U1.1 (SwC)
Other:
- moved on the sheet: D1
Changed lines of the file:
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@@
-	)
-	(junction
-		(at 137.16 97.79)
-		(diameter 0)
-		(color 0 0 0 0)
 	)
 	(junction
@@
 		(color 0 0 0 0)
 	)
+	(junction
+		(at 137.16 90.17)
+		(diameter 0)
+		(color 0 0 0 0)
+	)
+	(wire
+		(pts
+			(xy 134.62 97.79) (xy 134.62 90.17)
+		)
+		(stroke
+			(width 0)
+			(type default)
+		)
+	)
 	(wire
 		(pts
@@
 	(wire
 		(pts
-			(xy 130.81 97.79) (xy 137.16 97.79)
-		)
-		(stroke
-			(width 0)
-			(type default)
-		)
-	)
-	(wire
-		(pts
 			(xy 96.52 99.06) (xy 96.52 104.14)
 		)
@@
 	(wire
 		(pts
-			(xy 140.97 97.79) (xy 137.16 97.79)
+			(xy 140.97 100.33) (xy 137.16 100.33)
 		)
 		(stroke
@@
 	(wire
 		(pts
-			(xy 140.97 97.79) (xy 140.97 110.49)
+			(xy 140.97 100.33) (xy 140.97 110.49)
 		)
 		(stroke
@@
 	(wire
 		(pts
+			(xy 130.81 97.79) (xy 134.62 97.79)
+		)
+		(stroke
+			(width 0)
+			(type default)
+		)
+	)
+	(wire
+		(pts
 			(xy 96.52 92.71) (xy 96.52 93.98)
 		)
@@
 	(wire
 		(pts
+			(xy 134.62 90.17) (xy 137.16 90.17)
+		)
+		(stroke
+			(width 0)
+			(type default)
+		)
+	)
+	(wire
+		(pts
 			(xy 96.52 85.09) (xy 130.81 85.09)
 		)
@@
 		(pts
 			(xy 96.52 82.55) (xy 96.52 85.09)
+		)
+		(stroke
+			(width 0)
+			(type default)
+		)
+	)
+	(wire
+		(pts
+			(xy 137.16 92.71) (xy 137.16 90.17)
 		)
 		(stroke
@@
 	(symbol
 		(lib_id "Diode:1N5819")
-		(at 137.16 93.98 90)
+		(at 137.16 96.52 90)
 		(unit 1)
 		(body_style 1)
@@
 		(fields_autoplaced yes)
 		(property "Reference" "D1"
-			(at 139.7 93.0274 90)
+			(at 139.7 95.5674 90)
 			(show_name no)
 			(do_not_autoplace no)
@@
 		)
 		(property "Value" "1N5819"
-			(at 139.7 95.5674 90)
+			(at 139.7 98.1074 90)
 			(show_name no)
 			(do_not_autoplace no)
@@
 		)
 		(property "Footprint" "Diode_THT:D_DO-41_SOD81_P10.16mm_Horizontal"
-			(at 141.605 93.98 0)
+			(at 141.605 96.52 0)
 			(hide yes)
 			(show_name no)
@@
 		)
 		(property "Datasheet" "http://www.vishay.com/docs/88525/1n5817.pdf"
-			(at 137.16 93.98 0)
+			(at 137.16 96.52 0)
 			(hide yes)
 			(show_name no)
@@
 		)
 		(property "Description" "40V 1A Schottky Barrier Rectifier Diode, DO-41"
-			(at 137.16 93.98 0)
-			(hide yes)
-			(show_name no)
+			(at 137.16 96.52 0)
+			(hide yes)
+			(show_name no)
